File: eicon-diva-sch/eicon-diva-sch.sch (KiCad schematic (older format))
At the start: 23 parts, among them Q201 12c00, U201 24C32N, U202 AN2135SC

Commit message: sch: small fixes
Parts:
- gave numbers to parts that had none: 1
Changed lines of the file:
@@
 $EndComp
 $Comp
-L Connector:USB_B J?
+L Connector:USB_B JP101
 U 1 1 61046281
 P 2400 1950
-F 0 "J?" H 2457 2417 50  0000 C CNN
+F 0 "JP101" H 2457 2417 50  0000 C CNN
 F 1 "USB_B" H 2457 2326 50  0000 C CNN
 F 2 "" H 2550 1900 50  0001 C CNN
@@
 $EndComp
 Wire Wire Line
-	4850 2200 4850 2350
-Wire Wire Line
-	4950 2200 4950 2650
+	4950 2200 4950 2350
 Wire Wire Line
 	5050 2200 5050 2450
@@
 Wire Wire Line
 	6000 1800 6000 2350
-Wire Wire Line
-	6000 2350 4850 2350
-Connection ~ 4850 2350
-Wire Wire Line
-	4850 2350 4850 2650
 $Comp
 L power:+3.3V #PWR?
@@
 Text Notes 2800 2850 0    50   ~ 0
 U104
+Wire Wire Line
+	4850 2200 4850 2650
+Wire Wire Line
+	6000 2350 4950 2350
+Connection ~ 4950 2350
+Wire Wire Line
+	4950 2350 4950 2650
 $EndSCHEMATC
